Commit message: [perception] tracker, model loading

File: tbf_gripper_perception/urdf/exp.urdf.xacro (robot description, xacro)
@@ -9,4 +9,4 @@
   <xtion_camera name="camera" parent="base_link"
                 xyz="0  0  0.1" rpy="0 0 0"/>
-  <marker_macro id="5" parent="base_link" xyz="0 0 0.5" rpy="0 0 0" size="0.1" />
+  <!--<marker_macro id="5" parent="base_link" xyz="0 0 0.5" rpy="0 0 0" size="0.1" />-->
 </robot>

File: tbf_gripper_perception/urdf/marker_macro.urdf.xacro (robot description, xacro)
@@ -15,5 +15,6 @@
                 <origin xyz="0 0 0.000" rpy="0 0 0"/>
                 <geometry>
-                    <mesh filename="package://tbf_gripper_perception/meshes/marker_v2.dae" scale="${size} ${size} ${size}"/>
+                    <mesh filename="package://tbf_gripper_perception/meshes/marker_v2.dae"
+                          scale="${size} ${size} ${size}"/>
                 </geometry>
                 <material name="Greenish_marker">

File: tbf_gripper_perception/urdf/wlanbox_model.urdf.xacro (robot description, xacro)
@@ -2,5 +2,18 @@
 <robot xmlns:xacro="http://ros.org/wiki/xacro" name="wlanbox">
   <property name="M_PI" value="3.1415926535897931"/>
-  <link name="wlanbox_base_link">
+  <property name="MODEL_BASE_NAME" value="wlanbox_base_link"/>
+  <link name="${MODEL_BASE_NAME}">
+    <visual>
+      <origin xyz="0 0 0.000" rpy="0 0 0"/>
+      <geometry>
+        <mesh filename="package://tbf_gripper_perception/meshes/wlan_box.stl" scale="1e-3 1e-3 1e-3"/>
+      </geometry>
+      <material name="Greenish_marker">
+        <color rgba="0.3 0.7 0.3 1"/>
+      </material>
+    </visual>
   </link>
+  <xacro:include filename="$(find tbf_gripper_perception)/urdf/marker_macro.urdf.xacro"/>
+  <marker_macro id="50" parent="${MODEL_BASE_NAME}" xyz="0 0 0.078" rpy="0 0 0" size="0.08" />
+  <!--<marker_macro id="52" parent="foo" xyz="0 0 0.078" rpy="0 0 0" size="0.08" />-->
 </robot>

Commit message: [perception] full model tracking, basics working, no pose smoothing yet

File: tbf_gripper_perception/urdf/exp.urdf.xacro (robot description, xacro)
@@ -10,3 +10,9 @@
                 xyz="0  0  0.1" rpy="0 0 0"/>
   <!--<marker_macro id="5" parent="base_link" xyz="0 0 0.5" rpy="0 0 0" size="0.1" />-->
+  <joint name="wlanbox_float_joint" type="floating">
+    <origin xyz="0 0 0.5" rpy="0 0 0"/>
+    <parent link="base_link"/>
+    <child link="wlanbox_base_link"/>
+ </joint>
+  <xacro:include filename="$(find tbf_gripper_perception)/urdf/wlanbox_model.urdf.xacro"/>
 </robot>

File: tbf_gripper_perception/urdf/wlanbox_model.urdf.xacro (robot description, xacro)
@@ -15,5 +15,11 @@
   </link>
   <xacro:include filename="$(find tbf_gripper_perception)/urdf/marker_macro.urdf.xacro"/>
-  <marker_macro id="50" parent="${MODEL_BASE_NAME}" xyz="0 0 0.078" rpy="0 0 0" size="0.08" />
+  <marker_macro id="50" parent="${MODEL_BASE_NAME}" xyz="0 0 0.078" rpy="0 0 ${-0.5*M_PI}" size="0.08" />
+  <marker_macro id="53" parent="${MODEL_BASE_NAME}" xyz="-0.070 0.034 0.078" rpy="0 0 0" size="0.036" />
+  <marker_macro id="54" parent="${MODEL_BASE_NAME}" xyz="0.070 0.034 0.078" rpy="0 0 ${M_PI}" size="0.036" />
+  <marker_macro id="51" parent="${MODEL_BASE_NAME}" xyz="0.070 -0.034 0.078" rpy="0 0 ${M_PI}" size="0.036" />
+  <marker_macro id="52" parent="${MODEL_BASE_NAME}" xyz="-0.070 -0.034 0.078" rpy="0 0 0" size="0.036" />
+  <marker_macro id="55" parent="${MODEL_BASE_NAME}" xyz="0.050 ${0.12*0.5} 0.038" rpy="${-0.5*M_PI} ${-0.5*M_PI} 0" size="0.056" />
+  <marker_macro id="56" parent="${MODEL_BASE_NAME}" xyz="-0.052 ${0.12*0.5} 0.038" rpy="${-0.5*M_PI} ${-0.5*M_PI} 0" size="0.056" />
   <!--<marker_macro id="52" parent="foo" xyz="0 0 0.078" rpy="0 0 0" size="0.08" />-->
 </robot>
